File: PCB/breakout.kicad_pcb (KiCad board)
At the start: 2 copper layers, 25.4 x 17.8 mm, 21 parts, among them J1 BKOUT_PINS, J2 POTENTIOMETER, U1 AD5293

Commit message: update jumper solder mask
Other:
- board text added: "2023-04-21 2.0.2"
- board text removed: "2023-04-20 2.0.2"
Changed lines of the file:
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@@
   (title_block
     (title "AD5293_breakout")
-    (date "2023-04-20")
+    (date "2023-04-21")
     (rev "2.0.2")
     (company "Cedar Grove Studios")
@@
     (property "Sheetname" "")
     (attr exclude_from_pos_files)
-    (fp_text reference "JP1" (at -2.15 0.8) (layer "B.SilkS") hide
+    (fp_text reference "JP1" (at -2.15 0.8 180) (layer "B.SilkS") hide
       (effects (font (size 0.5 0.5) (thickness 0.1)) (justify mirror))
     )
-    (fp_text value "SDO PULL-UP" (at -5.1 0.05) (layer "B.SilkS")
+    (fp_text value "SDO PULL-UP" (at -5.1 0.05 180) (layer "B.SilkS")
       (effects (font (size 0.6 0.6) (thickness 0.1)) (justify mirror))
     )
@@
     (fp_arc (start -1.4 -0.3) (mid -1.194975 -0.794975) (end -0.7 -1) (layer "B.SilkS") (width 0.12))
     (fp_arc (start 1.4 0.3) (mid 1.194975 0.794975) (end 0.7 1) (layer "B.SilkS") (width 0.12))
+    (fp_rect (start -0.3 0.35) (end 0.3 -0.35) (layer "B.Mask") (width 0.01) (fill solid))
     (fp_line (start -1.65 1.25) (end 1.65 1.25) (layer "B.CrtYd") (width 0.05))
     (fp_line (start 1.65 -1.25) (end 1.65 1.25) (layer "B.CrtYd") (width 0.05))
     (fp_line (start 1.65 -1.25) (end -1.65 -1.25) (layer "B.CrtYd") (width 0.05))
     (fp_line (start -1.65 1.25) (end -1.65 -1.25) (layer "B.CrtYd") (width 0.05))
-    (pad "1" smd custom locked (at -0.65 0) (size 1 0.5) (layers "B.Cu" "B.Mask")
+    (pad "1" smd custom (at -0.65 0) (size 1 0.5) (layers "B.Cu" "B.Mask")
       (net 18 "Net-(JP1-Pad1)") (pinfunction "A") (pintype "passive") (zone_connect 2)
       (options (clearance outline) (anchor rect))
@@
           ) (width 0) (fill yes))
       ))
-    (pad "2" smd custom locked (at 0.65 0) (size 1 0.5) (layers "B.Cu" "B.Mask")
+    (pad "2" smd custom (at 0.65 0) (size 1 0.5) (layers "B.Cu" "B.Mask")
       (net 12 "/SDO") (pinfunction "B") (pintype "passive") (zone_connect 2)
       (options (clearance outline) (anchor rect))
@@
     (effects (font (size 0.6 0.6) (thickness 0.12) italic) (justify mirror))
   )
-  (gr_text "2023-04-20 2.0.2" (at 143.8 104.3) (layer "B.SilkS")
+  (gr_text "2023-04-21 2.0.2" (at 143.8 104.3) (layer "B.SilkS")
     (effects (font (size 0.5 0.5) (thickness 0.1)) (justify mirror))
   )
